File: hardware/v1/xt-at-pc-rgb-led-v1.kicad_sch (KiCad schematic)
At the start: 16 parts, among them J1 PLED, J2 HDD, J3 TURBO, J4 RGB LED (A R G B), J5 SW IN, J6 SW OUT, Q1 BC547, Q2 BC547

Commit message: Lay resistors and diodes flat on both boards
7.62 mm horizontal footprints, side by side; mounting holes in gaps
between the parts. v1 44 x 25.5 mm, v2 42 x 36.4 mm. Component height
about 8.5 mm.

Co-Authored-By: Claude Opus 5.5 (1M context) <noreply@anthropic.com>
Claude-Session: https://claude.ai/code/session_01JRatMm8Q7Nvo5CN8dD4gBk
Parts:
- D1, D2, D3, D4, D5: footprint Diode_THT:D_DO-35_SOD27_P2.54mm_Vertical_AnodeUp -> Diode_THT:D_DO-35_SOD27_P7.62mm_Horizontal
- R0, R1, R2: footprint Resistor_THT:R_Axial_DIN0207_L6.3mm_D2.5mm_P2.54mm_Vertical -> Resistor_THT:R_Axial_DIN0207_L6.3mm_D2.5mm_P7.62mm_Horizontal
Changed lines of the file:
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@@
     (instances
       (project "xt-at-pc-rgb-led-v1"
-        (path "/728e3474-736f-4dfe-b7de-60e4d1289106"
+        (path "/18e89ad3-a9bb-4d8b-ac46-a8cfacece97a"
           (reference "J1")
           (unit 1)))))
@@
     (instances
       (project "xt-at-pc-rgb-led-v1"
-        (path "/728e3474-736f-4dfe-b7de-60e4d1289106"
+        (path "/18e89ad3-a9bb-4d8b-ac46-a8cfacece97a"
           (reference "#PWR01")
           (unit 1)))))
@@
     (instances
       (project "xt-at-pc-rgb-led-v1"
-        (path "/728e3474-736f-4dfe-b7de-60e4d1289106"
+        (path "/18e89ad3-a9bb-4d8b-ac46-a8cfacece97a"
           (reference "J2")
           (unit 1)))))
@@
     (instances
       (project "xt-at-pc-rgb-led-v1"
-        (path "/728e3474-736f-4dfe-b7de-60e4d1289106"
+        (path "/18e89ad3-a9bb-4d8b-ac46-a8cfacece97a"
           (reference "J3")
           (unit 1)))))
@@
     (instances
       (project "xt-at-pc-rgb-led-v1"
-        (path "/728e3474-736f-4dfe-b7de-60e4d1289106"
+        (path "/18e89ad3-a9bb-4d8b-ac46-a8cfacece97a"
           (reference "J4")
           (unit 1)))))
@@
     (instances
       (project "xt-at-pc-rgb-led-v1"
-        (path "/728e3474-736f-4dfe-b7de-60e4d1289106"
+        (path "/18e89ad3-a9bb-4d8b-ac46-a8cfacece97a"
           (reference "J5")
           (unit 1)))))
@@
     (instances
       (project "xt-at-pc-rgb-led-v1"
-        (path "/728e3474-736f-4dfe-b7de-60e4d1289106"
+        (path "/18e89ad3-a9bb-4d8b-ac46-a8cfacece97a"
           (reference "J6")
           (unit 1)))))
@@
           (size 1.27 1.27))
         (justify left)))
-    (property "Footprint" "Resistor_THT:R_Axial_DIN0207_L6.3mm_D2.5mm_P2.54mm_Vertical"
+    (property "Footprint" "Resistor_THT:R_Axial_DIN0207_L6.3mm_D2.5mm_P7.62mm_Horizontal"
       (at 80 40 0)
       (effects
@@
     (instances
       (project "xt-at-pc-rgb-led-v1"
-        (path "/728e3474-736f-4dfe-b7de-60e4d1289106"
+        (path "/18e89ad3-a9bb-4d8b-ac46-a8cfacece97a"
           (reference "R0")
           (unit 1)))))
@@
           (size 1.27 1.27))
         (justify left)))
-    (property "Footprint" "Resistor_THT:R_Axial_DIN0207_L6.3mm_D2.5mm_P2.54mm_Vertical"
+    (property "Footprint" "Resistor_THT:R_Axial_DIN0207_L6.3mm_D2.5mm_P7.62mm_Horizontal"
       (at 110 40 0)
       (effects
@@
     (instances
       (project "xt-at-pc-rgb-led-v1"
-        (path "/728e3474-736f-4dfe-b7de-60e4d1289106"
+        (path "/18e89ad3-a9bb-4d8b-ac46-a8cfacece97a"
           (reference "R1")
           (unit 1)))))
@@
           (size 1.27 1.27))
         (justify left)))
-    (property "Footprint" "Resistor_THT:R_Axial_DIN0207_L6.3mm_D2.5mm_P2.54mm_Vertical"
+    (property "Footprint" "Resistor_THT:R_Axial_DIN0207_L6.3mm_D2.5mm_P7.62mm_Horizontal"
       (at 170 40 0)
       (effects
@@
     (instances
       (project "xt-at-pc-rgb-led-v1"
-        (path "/728e3474-736f-4dfe-b7de-60e4d1289106"
+        (path "/18e89ad3-a9bb-4d8b-ac46-a8cfacece97a"
           (reference "R2")
           (unit 1)))))
@@
     (instances
       (project "xt-at-pc-rgb-led-v1"
-        (path "/728e3474-736f-4dfe-b7de-60e4d1289106"
+        (path "/18e89ad3-a9bb-4d8b-ac46-a8cfacece97a"
           (reference "Q1")
           (unit 1)))))
@@
     (instances
       (project "xt-at-pc-rgb-led-v1"
-        (path "/728e3474-736f-4dfe-b7de-60e4d1289106"
+        (path "/18e89ad3-a9bb-4d8b-ac46-a8cfacece97a"
           (reference "Q2")
           (unit 1)))))
@@
         (font
           (size 1.27 1.27))))
-    (property "Footprint" "Diode_THT:D_DO-35_SOD27_P2.54mm_Vertical_AnodeUp"
+    (property "Footprint" "Diode_THT:D_DO-35_SOD27_P7.62mm_Horizontal"
       (at 100 130 0)
       (effects
@@
     (instances
       (project "xt-at-pc-rgb-led-v1"
-        (path "/728e3474-736f-4dfe-b7de-60e4d1289106"
+        (path "/18e89ad3-a9bb-4d8b-ac46-a8cfacece97a"
           (reference "D1")
           (unit 1)))))
@@
         (font
           (size 1.27 1.27))))
-    (property "Footprint" "Diode_THT:D_DO-35_SOD27_P2.54mm_Vertical_AnodeUp"
+    (property "Footprint" "Diode_THT:D_DO-35_SOD27_P7.62mm_Horizontal"
       (at 115 130 0)
       (effects
@@
     (instances
       (project "xt-at-pc-rgb-led-v1"
-        (path "/728e3474-736f-4dfe-b7de-60e4d1289106"
+        (path "/18e89ad3-a9bb-4d8b-ac46-a8cfacece97a"
           (reference "D2")
           (unit 1)))))
@@
         (font
           (size 1.27 1.27))))
-    (property "Footprint" "Diode_THT:D_DO-35_SOD27_P2.54mm_Vertical_AnodeUp"
+    (property "Footprint" "Diode_THT:D_DO-35_SOD27_P7.62mm_Horizontal"
       (at 160 130 0)
       (effects
@@
     (instances
       (project "xt-at-pc-rgb-led-v1"
-        (path "/728e3474-736f-4dfe-b7de-60e4d1289106"
+        (path "/18e89ad3-a9bb-4d8b-ac46-a8cfacece97a"
           (reference "D3")
           (unit 1)))))
@@
         (font
           (size 1.27 1.27))))
-    (property "Footprint" "Diode_THT:D_DO-35_SOD27_P2.54mm_Vertical_AnodeUp"
+    (property "Footprint" "Diode_THT:D_DO-35_SOD27_P7.62mm_Horizontal"
       (at 130 130 0)
       (effects
@@
     (instances
       (project "xt-at-pc-rgb-led-v1"
-        (path "/728e3474-736f-4dfe-b7de-60e4d1289106"
+        (path "/18e89ad3-a9bb-4d8b-ac46-a8cfacece97a"
           (reference "D4")
           (unit 1)))))
@@
     (instances
       (project "xt-at-pc-rgb-led-v1"
-        (path "/728e3474-736f-4dfe-b7de-60e4d1289106"
+        (path "/18e89ad3-a9bb-4d8b-ac46-a8cfacece97a"
           (reference "#PWR02")
           (unit 1)))))
@@
         (font
           (size 1.27 1.27))))
-    (property "Footprint" "Diode_THT:D_DO-35_SOD27_P2.54mm_Vertical_AnodeUp"
+    (property "Footprint" "Diode_THT:D_DO-35_SOD27_P7.62mm_Horizontal"
       (at 190 130 0)
       (effects
@@
     (instances
       (project "xt-at-pc-rgb-led-v1"
-        (path "/728e3474-736f-4dfe-b7de-60e4d1289106"
+        (path "/18e89ad3-a9bb-4d8b-ac46-a8cfacece97a"
           (reference "D5")
           (unit 1)))))
@@
     (instances
       (project "xt-at-pc-rgb-led-v1"
-        (path "/728e3474-736f-4dfe-b7de-60e4d1289106"
+        (path "/18e89ad3-a9bb-4d8b-ac46-a8cfacece97a"
           (reference "#FLG01")
           (unit 1)))))
@@
     (instances
       (project "xt-at-pc-rgb-led-v1"
-        (path "/728e3474-736f-4dfe-b7de-60e4d1289106"
+        (path "/18e89ad3-a9bb-4d8b-ac46-a8cfacece97a"
           (reference "#PWR04")
           (unit 1)))))
