File: hardware/v2/xt-at-pc-rgb-led-v2.kicad_sch (KiCad schematic)
At the start: 23 parts, among them J1 +5V GND, J2 HDD, J3 TURBO, J4 SW IN, J5 SW OUT, J6 ADDR LED (5V DATA GND), J7 RGB LED (COM R G B), J8 ISP, U1 ATtiny84A-PU

Commit message: Lay resistors and diodes flat on both boards
7.62 mm horizontal footprints, side by side; mounting holes in gaps
between the parts. v1 44 x 25.5 mm, v2 42 x 36.4 mm. Component height
about 8.5 mm.

Co-Authored-By: Claude Opus 5.5 (1M context) <noreply@anthropic.com>
Claude-Session: https://claude.ai/code/session_01JRatMm8Q7Nvo5CN8dD4gBk
Parts:
- R1, R10, R11, R2, R3, R4, R5, R6, R7, R8, R9: footprint Resistor_THT:R_Axial_DIN0207_L6.3mm_D2.5mm_P2.54mm_Vertical -> Resistor_THT:R_Axial_DIN0207_L6.3mm_D2.5mm_P7.62mm_Horizontal
